File: kicad/leafony_bus.kicad_sch (KiCad schematic)
At the start: 1 part, among them CN1 Leafony Bus

Commit message: BOMからCN1を除外
Parts:
- CN1: now left out of the parts list
Changed lines of the file:
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@@
 		(unit 1)
 		(exclude_from_sim no)
-		(in_bom yes)
+		(in_bom no)
 		(on_board yes)
 		(dnp no)
